File: dualpaneldriver/dualpaneldriver.sch (KiCad schematic (older format))
At the start: 7 parts

Commit message: some components placed
Parts:
- R101, R102, R103: footprint (none) -> Resistor_SMD:R_0603_1608Metric
Changed lines of the file:
@@
 F 0 "R103" H 3959 6396 50  0000 L CNN
 F 1 "200" H 3959 6305 50  0000 L CNN
-F 2 "" H 3900 6350 50  0001 C CNN
+F 2 "Resistor_SMD:R_0603_1608Metric" H 3900 6350 50  0001 C CNN
 F 3 "~" H 3900 6350 50  0001 C CNN
 	1    3900 6350
@@
 F 0 "R102" H 3959 4396 50  0000 L CNN
 F 1 "200" H 3959 4305 50  0000 L CNN
-F 2 "" H 3900 4350 50  0001 C CNN
+F 2 "Resistor_SMD:R_0603_1608Metric" H 3900 4350 50  0001 C CNN
 F 3 "~" H 3900 4350 50  0001 C CNN
 	1    3900 4350
@@
 F 0 "R101" H 3959 2396 50  0000 L CNN
 F 1 "200" H 3959 2305 50  0000 L CNN
-F 2 "" H 3900 2350 50  0001 C CNN
+F 2 "Resistor_SMD:R_0603_1608Metric" H 3900 2350 50  0001 C CNN
 F 3 "~" H 3900 2350 50  0001 C CNN
 	1    3900 2350

Commit message: i'm too sleepy to continue
Parts:
- removed H102: M3, MountingHole:MountingHole_3.2mm_M3_ISO7380_Pad, symbol Mechanical:MountingHole_Pad
- G101: footprint Automated:fully_automated_logo_soldermask -> Automated:falogo_small_copper
Connections:
- no-connect marks 2 -> 1
Changed lines of the file:
@@
 NoConn ~ 850  7400
-$Comp
-L Mechanical:MountingHole_Pad H102
-U 1 1 5E17729B
-P 1250 7300
-F 0 "H102" H 1350 7349 50  0000 L CNN
-F 1 "M3" H 1350 7258 50  0000 L CNN
-F 2 "MountingHole:MountingHole_3.2mm_M3_ISO7380_Pad" H 1250 7300 50  0001 C CNN
-F 3 "~" H 1250 7300 50  0001 C CNN
-F 4 "d.n.p." H 1250 7300 50  0001 C CNN "V1"
-	1    1250 7300
-	1    0    0    -1
-$EndComp
-NoConn ~ 1250 7400
 $Comp
 L meansOfCircuitDesign:Fully_Automated_Logo G101
@@
 F 0 "G101" H 1150 6350 60  0001 C CNN
 F 1 "Fully_Automated_Logo" H 1050 6890 60  0001 C CNN
-F 2 "Automated:fully_automated_logo_soldermask" H 1050 6600 50  0001 C CNN
+F 2 "Automated:falogo_small_copper" H 1050 6600 50  0001 C CNN
 F 3 "" H 1050 6600 50  0001 C CNN
 F 4 "d.n.p." H 1050 6600 50  0001 C CNN "V1"
@@
 L Graphic:SYM_Arrow45_Large G102
 U 1 1 5E17963F
-P 1750 7300
-F 0 "G102" H 1750 7460 50  0001 C CNN
-F 1 "Transsistor Logo" H 2050 7050 50  0000 R CNN
-F 2 "Automated:transistor_10x10mm" H 1750 7300 50  0001 C CNN
-F 3 "~" H 1750 7300 50  0001 C CNN
-F 4 "d.n.p." H 1750 7300 50  0001 C CNN "V1"
-	1    1750 7300
+P 1450 7250
+F 0 "G102" H 1450 7410 50  0001 C CNN
+F 1 "Transsistor Logo" H 1750 7000 50  0000 R CNN
+F 2 "Automated:transistor_10x10mm" H 1450 7250 50  0001 C CNN
+F 3 "~" H 1450 7250 50  0001 C CNN
+F 4 "d.n.p." H 1450 7250 50  0001 C CNN "V1"
+	1    1450 7250
 	-1   0    0    -1
 $EndComp
@@
 L Graphic:SYM_Arrow45_Large #SYM101
 U 1 1 5E17B2EC
-P 1700 7250
-F 0 "#SYM101" H 1700 7410 50  0001 C CNN
-F 1 "SYM_Arrow45_Large" H 1700 7110 50  0001 C CNN
-F 2 "" H 1700 7250 50  0001 C CNN
-F 3 "~" H 1700 7250 50  0001 C CNN
-	1    1700 7250
+P 1400 7200
+F 0 "#SYM101" H 1400 7360 50  0001 C CNN
+F 1 "SYM_Arrow45_Large" H 1400 7060 50  0001 C CNN
+F 2 "" H 1400 7200 50  0001 C CNN
+F 3 "~" H 1400 7200 50  0001 C CNN
+	1    1400 7200
 	0    1    1    0
 $EndComp
@@
 L Graphic:SYM_Arrow45_Large #SYM102
 U 1 1 5E17BE68
-P 1800 7350
-F 0 "#SYM102" H 1800 7510 50  0001 C CNN
-F 1 "SYM_Arrow45_Large" H 1800 7210 50  0001 C CNN
-F 2 "" H 1800 7350 50  0001 C CNN
-F 3 "~" H 1800 7350 50  0001 C CNN
-	1    1800 7350
+P 1500 7300
+F 0 "#SYM102" H 1500 7460 50  0001 C CNN
+F 1 "SYM_Arrow45_Large" H 1500 7160 50  0001 C CNN
+F 2 "" H 1500 7300 50  0001 C CNN
+F 3 "~" H 1500 7300 50  0001 C CNN
+	1    1500 7300
 	0    1    1    0
 $EndComp
