File: dualpaneldriver/microcontroller.sch (KiCad schematic (older format))
At the start: 57 parts, among them J401 PIR1, J402 Conn_01x02, J403 PIR2, J404 HALL, J405 PIR3, J406 WS2812CTRL, J407 I2C, J408 CAN, J409 Conn_ARM_JTAG_SWD_10, J410 UART, J411 CAN, Q401 AO3400, SW401 POWERON, U401 STM32F072C8Tx, U402 VEML3328, U403 OPT3001, U404 SN65HVD232, Y401 8.000MHz

Commit message: i'm too sleepy to continue
Parts:
- removed C408: 100nF, Capacitor_SMD:C_0603_1608Metric, symbol Device:C_Small
- added C413: 100nF, Capacitor_SMD:C_0603_1608Metric, symbol Device:C_Small
- added J412: POWERSW, Connector_PinHeader_2.54mm:PinHeader_1x02_P2.54mm_Vertical, symbol Connector_Generic:Conn_01x02
- added R420: 1k, Resistor_SMD:R_0603_1608Metric, symbol Device:R_Small
- added R421: 360k, Resistor_SMD:R_0603_1608Metric, symbol Device:R_Small
- added SW402: POWERON, Automated:SW_SPST_PTS636_G, symbol Switch:SW_Push
- J402: value Conn_01x02 -> USERSW
- SW401: value POWERON -> USER
Connections:
- net +3V3: now also R420.2
- net GNDD: now also C413.2, J412.2 (Pin_2), SW402.1
- net ADC_IN9 renamed WAKEUP_SW
- net WAKEUP_SW: now also C413.1, R421.2
- new net: J412.1 (Pin_1), R420.1, R421.1, SW402.2
Other:
- note added: "user\nbutton"
- note removed: "OPAMP"
- moved on the sheet: C409
Changed lines of the file:
@@
 Decoupling Caps
-$Comp
-L power:+5VL #PWR0415
-U 1 1 5DE17221
-P 4100 6750
-F 0 "#PWR0415" H 4100 6600 50  0001 C CNN
-F 1 "+5VL" H 4115 6923 50  0000 C CNN
-F 2 "" H 4100 6750 50  0001 C CNN
-F 3 "" H 4100 6750 50  0001 C CNN
-	1    4100 6750
-	1    0    0    -1
-$EndComp
-$Comp
-L Device:C_Small C?
-U 1 1 5DE1AA53
-P 4100 7000
-AR Path="/5DC023B6/5DE1AA53" Ref="C?"  Part="1"
-AR Path="/5DC65EA5/5DE1AA53" Ref="C?"  Part="1"
-AR Path="/5DC18E4B/5DE1AA53" Ref="C408"  Part="1"
-F 0 "C408" H 4192 7046 50  0000 L CNN
-F 1 "100nF" H 4192 6955 50  0000 L CNN
-F 2 "Capacitor_SMD:C_0603_1608Metric" H 4100 7000 50  0001 C CNN
-F 3 "~" H 4100 7000 50  0001 C CNN
-	1    4100 7000
-	1    0    0    -1
-$EndComp
-Wire Wire Line
-	4100 6900 4100 6750
 $Comp
 L Connector_Generic:Conn_01x04 J408
@@
 P 6900 2600
 F 0 "SW401" H 6900 2885 50  0000 C CNN
-F 1 "POWERON" H 6900 2794 50  0000 C CNN
+F 1 "USER" H 6900 2794 50  0000 C CNN
 F 2 "Automated:SW_SPST_PTS636_G" H 6900 2800 50  0001 C CNN
 F 3 "https://www.mouser.at/datasheet/2/60/pts636-1550567.pdf" H 6900 2800 50  0001 C CNN
@@
 Wire Wire Line
 	9650 1050 9900 1050
-Text Notes 6850 2850 0    50   ~ 0
+Text Notes 5100 2850 0    50   ~ 0
 power\nbutton
 Text Notes 2100 4300 2    50   ~ 0
@@
 AR Path="/5DC18E4B/5DD2193F" Ref="J402"  Part="1"
 F 0 "J402" H 6868 3367 50  0000 C CNN
-F 1 "Conn_01x02" H 6868 3276 50  0000 C CNN
+F 1 "USERSW" H 6868 3276 50  0000 C CNN
 F 2 "Connector_PinHeader_2.54mm:PinHeader_1x02_P2.54mm_Vertical" H 6950 3150 50  0001 C CNN
 F 3 "~" H 6950 3150 50  0001 C CNN
@@
 Wire Wire Line
 	2850 1150 2900 1150
-Text Label 1600 2750 0    50   ~ 0
-ADC_IN9
-Text Notes 4000 6500 0    50   ~ 0
-OPAMP
-$Comp
-L power:GNDA #PWR0416
-U 1 1 5E00AECE
-P 4100 7250
-F 0 "#PWR0416" H 4100 7000 50  0001 C CNN
-F 1 "GNDA" H 4105 7077 50  0000 C CNN
-F 2 "" H 4100 7250 50  0001 C CNN
-F 3 "" H 4100 7250 50  0001 C CNN
-	1    4100 7250
-	1    0    0    -1
-$EndComp
-Wire Wire Line
-	4100 7250 4100 7100
 $Comp
 L Device:C_Small C?
 U 1 1 5E069A31
-P 4550 7000
+P 4050 7000
 AR Path="/5DC023B6/5E069A31" Ref="C?"  Part="1"
 AR Path="/5DC65EA5/5E069A31" Ref="C?"  Part="1"
 AR Path="/5DC18E4B/5E069A31" Ref="C409"  Part="1"
-F 0 "C409" H 4642 7046 50  0000 L CNN
-F 1 "100nF" H 4642 6955 50  0000 L CNN
-F 2 "Capacitor_SMD:C_0603_1608Metric" H 4550 7000 50  0001 C CNN
-F 3 "~" H 4550 7000 50  0001 C CNN
-	1    4550 7000
+F 0 "C409" H 4142 7046 50  0000 L CNN
+F 1 "100nF" H 4142 6955 50  0000 L CNN
+F 2 "Capacitor_SMD:C_0603_1608Metric" H 4050 7000 50  0001 C CNN
+F 3 "~" H 4050 7000 50  0001 C CNN
+	1    4050 7000
 	1    0    0    -1
 $EndComp
@@
 L power:GNDD #PWR0418
 U 1 1 5E06A0B0
-P 4550 7250
-F 0 "#PWR0418" H 4550 7000 50  0001 C CNN
-F 1 "GNDD" H 4554 7095 50  0000 C CNN
-F 2 "" H 4550 7250 50  0001 C CNN
-F 3 "" H 4550 7250 50  0001 C CNN
-	1    4550 7250
-	1    0    0    -1
-$EndComp
-Wire Wire Line
-	4550 7250 4550 7100
+P 4050 7250
+F 0 "#PWR0418" H 4050 7000 50  0001 C CNN
+F 1 "GNDD" H 4054 7095 50  0000 C CNN
+F 2 "" H 4050 7250 50  0001 C CNN
+F 3 "" H 4050 7250 50  0001 C CNN
+	1    4050 7250
+	1    0    0    -1
+$EndComp
+Wire Wire Line
+	4050 7250 4050 7100
 $Comp
 L power:+3.3V #PWR0417
 U 1 1 5E0B6973
-P 4550 6750
-F 0 "#PWR0417" H 4550 6600 50  0001 C CNN
-F 1 "+3.3V" H 4565 6923 50  0000 C CNN
-F 2 "" H 4550 6750 50  0001 C CNN
-F 3 "" H 4550 6750 50  0001 C CNN
-	1    4550 6750
-	1    0    0    -1
-$EndComp
-Wire Wire Line
-	4550 6750 4550 6900
+P 4050 6750
+F 0 "#PWR0417" H 4050 6600 50  0001 C CNN
+F 1 "+3.3V" H 4065 6923 50  0000 C CNN
+F 2 "" H 4050 6750 50  0001 C CNN
+F 3 "" H 4050 6750 50  0001 C CNN
+	1    4050 6750
+	1    0    0    -1
+$EndComp
+Wire Wire Line
+	4050 6750 4050 6900
 Wire Wire Line
 	6650 4000 6950 4000
@@
 Text Label 6700 5350 2    50   ~ 0
 I2C_SCL
+$Comp
+L Switch:SW_Push SW402
+U 1 1 5DE67F91
+P 5200 2600
+F 0 "SW402" H 5200 2885 50  0000 C CNN
+F 1 "POWERON" H 5200 2794 50  0000 C CNN
+F 2 "Automated:SW_SPST_PTS636_G" H 5200 2800 50  0001 C CNN
+F 3 "https://www.mouser.at/datasheet/2/60/pts636-1550567.pdf" H 5200 2800 50  0001 C CNN
+F 4 "PTS636-SP43-SMTR-LFS" H 5200 2600 50  0001 C CNN "V1"
+	1    5200 2600
+	1    0    0    -1
+$EndComp
+$Comp
+L power:GNDD #PWR0458
+U 1 1 5DE67F98
+P 5900 2900
+F 0 "#PWR0458" H 5900 2650 50  0001 C CNN
+F 1 "GNDD" H 5904 2745 50  0000 C CNN
+F 2 "" H 5900 2900 50  0001 C CNN
+F 3 "" H 5900 2900 50  0001 C CNN
+	1    5900 2900
+	1    0    0    -1
+$EndComp
+$Comp
+L Device:C_Small C?
+U 1 1 5DE67F9E
+P 5900 2750
+AR Path="/5DC023B6/5DE67F9E" Ref="C?"  Part="1"
+AR Path="/5DC65EA5/5DE67F9E" Ref="C?"  Part="1"
+AR Path="/5DC18E4B/5DE67F9E" Ref="C413"  Part="1"
+F 0 "C413" H 5992 2796 50  0000 L CNN
+F 1 "100nF" H 5992 2705 50  0000 L CNN
+F 2 "Capacitor_SMD:C_0603_1608Metric" H 5900 2750 50  0001 C CNN
+F 3 "~" H 5900 2750 50  0001 C CNN
+	1    5900 2750
+	1    0    0    -1
+$EndComp
+Wire Wire Line
+	5900 2850 5900 2900
+Wire Wire Line
+	5900 2650 5900 2600
+Connection ~ 5900 2600
+Wire Wire Line
+	5900 2600 6450 2600
+$Comp
+L Device:R_Small R?
+U 1 1 5DE67FA9
+P 5700 2600
+AR Path="/5DC023B6/5DE67FA9" Ref="R?"  Part="1"
+AR Path="/5DC65EA5/5DE67FA9" Ref="R?"  Part="1"
+AR Path="/5DC18E4B/5DE67FA9" Ref="R421"  Part="1"
+F 0 "R421" V 5596 2600 50  0000 C CNN
+F 1 "360k" V 5505 2600 50  0000 C CNN
+F 2 "Resistor_SMD:R_0603_1608Metric" H 5700 2600 50  0001 C CNN
+F 3 "~" H 5700 2600 50  0001 C CNN
+F 4 "" H 5700 2600 50  0001 C CNN "V1"
+	1    5700 2600
+	0    -1   -1   0
+$EndComp
+Wire Wire Line
+	5800 2600 5900 2600
+Wire Wire Line
+	5600 2600 5500 2600
+$Comp
+L power:GNDD #PWR0455
+U 1 1 5DE67FB1
+P 4950 2650
+F 0 "#PWR0455" H 4950 2400 50  0001 C CNN
+F 1 "GNDD" H 4954 2495 50  0000 C CNN
+F 2 "" H 4950 2650 50  0001 C CNN
+F 3 "" H 4950 2650 50  0001 C CNN
+	1    4950 2650
+	1    0    0    -1
+$EndComp
+Wire Wire Line
+	4950 2650 4950 2600
+Wire Wire Line
+	4950 2600 5000 2600
+$Comp
+L power:+3.3V #PWR0456
+U 1 1 5DE67FB9
+P 5450 2350
+F 0 "#PWR0456" H 5450 2200 50  0001 C CNN
+F 1 "+3.3V" H 5465 2523 50  0000 C CNN
+F 2 "" H 5450 2350 50  0001 C CNN
+F 3 "" H 5450 2350 50  0001 C CNN
+	1    5450 2350
+	1    0    0    -1
+$EndComp
+$Comp
+L Device:R_Small R420
+U 1 1 5DE67FBF
+P 5450 2450
+F 0 "R420" H 5391 2404 50  0000 R CNN
+F 1 "1k" H 5391 2495 50  0000 R CNN
+F 2 "Resistor_SMD:R_0603_1608Metric" H 5450 2450 50  0001 C CNN
+F 3 "~" H 5450 2450 50  0001 C CNN
+	1    5450 2450
+	-1   0    0    1
+$EndComp
+Wire Wire Line
+	5450 2550 5450 2600
+Connection ~ 5450 2600
+Wire Wire Line
+	5450 2600 5400 2600
+Text Notes 6800 2850 0    50   ~ 0
+user\nbutton
+$Comp
+L Connector_Generic:Conn_01x02 J?
+U 1 1 5DE67FC9
+P 5250 3150
+AR Path="/5DC18DED/5DE67FC9" Ref="J?"  Part="1"
+AR Path="/5DC18EA6/5DE67FC9" Ref="J?"  Part="1"
+AR Path="/5DC91BAA/5DE67FC9" Ref="J?"  Part="1"
+AR Path="/5DC18E4B/5DE67FC9" Ref="J412"  Part="1"
+F 0 "J412" H 5168 3367 50  0000 C CNN
+F 1 "POWERSW" H 5168 3276 50  0000 C CNN
+F 2 "Connector_PinHeader_2.54mm:PinHeader_1x02_P2.54mm_Vertical" H 5250 3150 50  0001 C CNN
+F 3 "~" H 5250 3150 50  0001 C CNN
+	1    5250 3150
+	-1   0    0    -1
+$EndComp
+Wire Wire Line
+	5450 3150 5500 3150
+Wire Wire Line
+	5500 3150 5500 2600
+Connection ~ 5500 2600
+Wire Wire Line
+	5500 2600 5450 2600
+$Comp
+L power:GNDD #PWR0457
+U 1 1 5DE67FD3
+P 5500 3300
+F 0 "#PWR0457" H 5500 3050 50  0001 C CNN
+F 1 "GNDD" H 5504 3145 50  0000 C CNN
+F 2 "" H 5500 3300 50  0001 C CNN
+F 3 "" H 5500 3300 50  0001 C CNN
+	1    5500 3300
+	1    0    0    -1
+$EndComp
+Wire Wire Line
+	5500 3300 5500 3250
+Wire Wire Line
+	5500 3250 5450 3250
+Text Label 6450 2600 2    50   ~ 0
+WAKEUP_SW
+Text Label 1600 2750 0    50   ~ 0
+WAKEUP_SW
 $EndSCHEMATC

Commit message: 100% routed, silkscreen still fucked up
Parts:
- J401: value PIR1 -> PIR3
- J405: value PIR3 -> PIR1
Connections:
- net MOTION1: now also R413.2; no longer R406.2
- net MOTION3: now also R406.2; no longer R413.2
Changed lines of the file:
@@
 P 8700 1100
 F 0 "J405" H 8780 1142 50  0000 L CNN
-F 1 "PIR3" H 8780 1051 50  0000 L CNN
+F 1 "PIR1" H 8780 1051 50  0000 L CNN
 F 2 "Connector_PinHeader_2.54mm:PinHeader_1x03_P2.54mm_Vertical" H 8700 1100 50  0001 C CNN
 F 3 "~" H 8700 1100 50  0001 C CNN
@@
 Wire Wire Line
 	8500 1100 8400 1100
-Text Label 5400 1100 0    50   ~ 0
+Text Label 7850 1100 0    50   ~ 0
 MOTION1
 $Comp
@@
 P 6250 1100
 F 0 "J401" H 6330 1142 50  0000 L CNN
-F 1 "PIR1" H 6330 1051 50  0000 L CNN
+F 1 "PIR3" H 6330 1051 50  0000 L CNN
 F 2 "Connector_PinHeader_2.54mm:PinHeader_1x03_P2.54mm_Vertical" H 6250 1100 50  0001 C CNN
 F 3 "~" H 6250 1100 50  0001 C CNN
@@
 Wire Wire Line
 	6050 1100 5950 1100
-Text Label 7850 1100 0    50   ~ 0
+Text Label 5400 1100 0    50   ~ 0
 MOTION3
 $Comp
