File: sevenSegmentClock/sevenSegmentClock.kicad_pcb (KiCad board)
At the start: 2 copper layers, 94 x 18 mm, 10 parts, among them J101 Conn_01x03, J102 Conn_01x03, J103 Conn_01x03, J104 Conn_01x03

Commit message: made the board chonky
Parts:
- added C1: 2.2uF/10V, Capacitor_SMD:C_0603_1608Metric, F.Cu at (240.8, 93.8)
- moved J103 13.0 mm to (244.3, 89.5)
- moved J104 13.0 mm to (247.1, 97.5)
- moved R101 13.0 mm to (242.2, 95.0)
- moved C101 11.5 mm to (184.0, 95.0)
- moved J101 11.5 mm to (184.0, 90.0)
- moved J102 11.5 mm to (181.5, 97.5)
- moved D103 10.5 mm to (235.5, 95.0)
- moved D101 9.50 mm to (193.5, 95.0)
- moved D102 0.50 mm to (214.5, 95.0)
Routing:
- net Net-(D102-Pad2): track 37.5 -> 27.1 mm
- net Net-(D101-Pad2): track 37.3 -> 27.1 mm
- net /DIN: track 24.1 -> 22.1 mm
- net +5V: track 4.92 -> 5.88 mm, vias 4 -> 5
Other:
- board size 94 x 18 mm -> 71 x 18 mm

Commit message: changed logo from silkscreen to solder mask
Parts:
- G101: footprint Automated:fully_automated_logo_silkscreen -> Automated:fully_automated_logo_soldermask
- moved G101 5.50 mm to (225.5, 95.0)

Commit message: added arrows and shit
Parts:
- added J1: Conn_01x01, TestPoint:TestPoint_THTPad_2.0x2.0mm_Drill1.0mm, F.Cu at (180.5, 95.0)
- added J2: Conn_01x01, TestPoint:TestPoint_THTPad_2.0x2.0mm_Drill1.0mm, F.Cu at (248.5, 95.0)
Routing:
- net /DIN: track 22.1 -> 96.4 mm
- net /DOUT: track 11.5 -> 85.2 mm
- net Net-(D101-Pad2): track 27.1 -> 26.0 mm
Other:
- board text added: "+5V DIN GND"
- board text added: "+5V DOUT GND"
- board text added: "G DIN +5V"
- board text added: "GND DOUT +5V"
- board text added: "IN"
- board text added: "JLCJLCJLCJLC"
- board text added: "O"
