File: sevenSegmentClock/sevenSegmentClock.sch (KiCad schematic (older format))
At the start: 10 parts, among them J101 Conn_01x03, J102 Conn_01x03, J103 Conn_01x03, J104 Conn_01x03

Commit message: made the board chonky
Parts:
- added C1: 2.2uF/10V, Capacitor_SMD:C_0603_1608Metric, symbol Device:C_Small
Connections:
- net +5V: now also C1.1
- net GND: now also C1.2
Changed lines of the file:
@@
 	1    0    0    -1
 $EndComp
+$Comp
+L Device:C_Small C1
+U 1 1 5EA87AF9
+P 1350 3900
+F 0 "C1" H 1442 3946 50  0000 L CNN
+F 1 "2.2uF/10V" H 1442 3855 50  0000 L CNN
+F 2 "Capacitor_SMD:C_0603_1608Metric" H 1350 3900 50  0001 C CNN
+F 3 "~" H 1350 3900 50  0001 C CNN
+	1    1350 3900
+	1    0    0    -1
+$EndComp
+$Comp
+L power:GND #PWR0113
+U 1 1 5EA87AFF
+P 1350 4000
+F 0 "#PWR0113" H 1350 3750 50  0001 C CNN
+F 1 "GND" H 1355 3827 50  0000 C CNN
+F 2 "" H 1350 4000 50  0001 C CNN
+F 3 "" H 1350 4000 50  0001 C CNN
+	1    1350 4000
+	-1   0    0    -1
+$EndComp
+$Comp
+L power:+5V #PWR0114
+U 1 1 5EA87B05
+P 1350 3800
+F 0 "#PWR0114" H 1350 3650 50  0001 C CNN
+F 1 "+5V" H 1365 3973 50  0000 C CNN
+F 2 "" H 1350 3800 50  0001 C CNN
+F 3 "" H 1350 3800 50  0001 C CNN
+	1    1350 3800
+	-1   0    0    -1
+$EndComp
 $EndSCHEMATC

Commit message: changed logo from silkscreen to solder mask
Parts:
- G101: footprint Automated:fully_automated_logo_silkscreen -> Automated:fully_automated_logo_soldermask
Changed lines of the file:
@@
 F 0 "G101" H 6400 6700 60  0001 C CNN
 F 1 "Fully_Automated_Logo" H 6300 7240 60  0001 C CNN
-F 2 "Automated:fully_automated_logo_silkscreen" H 6300 6950 50  0001 C CNN
+F 2 "Automated:fully_automated_logo_soldermask" H 6300 6950 50  0001 C CNN
 F 3 "" H 6300 6950 50  0001 C CNN
 	1    6300 6950

Commit message: added arrows and shit
Parts:
- added J1, J2: Conn_01x01, TestPoint:TestPoint_THTPad_1.5x1.5mm_Drill0.7mm, symbol Connector_Generic:Conn_01x01
Connections:
- net DIN: now also J2.1 (Pin_1)
- net DOUT: now also J1.1 (Pin_1)
Changed lines of the file:
@@
 DIN
 Wire Wire Line
-	2850 3250 3900 3250
+	2850 3250 3500 3250
 Connection ~ 2850 3250
 Wire Wire Line
@@
 $EndComp
 Wire Wire Line
-	8200 3250 8450 3250
+	8200 3250 8250 3250
 $Comp
 L meansOfCircuitDesign:Fully_Automated_Logo G101
@@
 	-1   0    0    -1
 $EndComp
+$Comp
+L Connector_Generic:Conn_01x01 J1
+U 1 1 5EA8E1A3
+P 2200 3900
+F 0 "J1" H 2118 3675 50  0000 C CNN
+F 1 "Conn_01x01" H 2118 3766 50  0000 C CNN
+F 2 "TestPoint:TestPoint_THTPad_1.5x1.5mm_Drill0.7mm" H 2200 3900 50  0001 C CNN
+F 3 "~" H 2200 3900 50  0001 C CNN
+	1    2200 3900
+	-1   0    0    1
+$EndComp
+Wire Wire Line
+	2400 3900 8250 3900
+Wire Wire Line
+	8250 3900 8250 3250
+Connection ~ 8250 3250
+Wire Wire Line
+	8250 3250 8450 3250
+$Comp
+L Connector_Generic:Conn_01x01 J2
+U 1 1 5EA9025F
+P 9100 2400
+F 0 "J2" H 9180 2442 50  0000 L CNN
+F 1 "Conn_01x01" H 9180 2351 50  0000 L CNN
+F 2 "TestPoint:TestPoint_THTPad_1.5x1.5mm_Drill0.7mm" H 9100 2400 50  0001 C CNN
+F 3 "~" H 9100 2400 50  0001 C CNN
+	1    9100 2400
+	1    0    0    -1
+$EndComp
+Wire Wire Line
+	8900 2400 3500 2400
+Wire Wire Line
+	3500 2400 3500 3250
+Connection ~ 3500 3250
+Wire Wire Line
+	3500 3250 3900 3250
 $EndSCHEMATC
